File: USB-EMI-Filter.kicad_pcb (KiCad board)
At the start: 2 copper layers, 51 x 18 mm, 12 parts, among them J1 USB_A, J2 USB_A, J3 CONN_01X02

Commit message: DRC, ERC passed
Other:
- rule via_min_size: 0.4 -> 0.6
Changed lines of the file:
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@@
   )
   (setup
-    (last_trace_width 1)
+    (last_trace_width 0.3)
     (user_trace_width 0.4)
     (user_trace_width 0.6)
@@
     (via_size 0.6)
     (via_drill 0.3)
-    (via_min_size 0.4)
+    (via_min_size 0.6)
     (via_min_drill 0.3)
     (uvia_size 0.3)
