File: USB-EMI-Filter.sch (KiCad schematic (older format))
At the start: 12 parts, among them J1 USB_A, J2 USB_A, J3 CONN_01X02

Commit message: DRC, ERC passed
Changed lines of the file:
@@
 EESchema Schematic File Version 4
+LIBS:USB-EMI-Filter-cache
 EELAYER 29 0
 EELAYER END
@@
 $EndComp
 Wire Wire Line
-	4025 3150 4625 3150
+	4025 3150 4375 3150
 Connection ~ 4625 3150
 $Comp
@@
 Connection ~ 7325 3150
 Wire Wire Line
-	7325 3150 7575 3150
+	7325 3150 7475 3150
 $Comp
 L power:GND #PWR0109
@@
 Wire Wire Line
 	7225 4275 7225 4300
+$Comp
+L power:PWR_FLAG #FLG0102
+U 1 1 5CABD24B
+P 4375 3150
+F 0 "#FLG0102" H 4375 3225 50  0001 C CNN
+F 1 "PWR_FLAG" H 4375 3323 50  0000 C CNN
+F 2 "" H 4375 3150 50  0001 C CNN
+F 3 "~" H 4375 3150 50  0001 C CNN
+	1    4375 3150
+	1    0    0    -1
+$EndComp
+Connection ~ 4375 3150
+Wire Wire Line
+	4375 3150 4625 3150
+$Comp
+L power:PWR_FLAG #FLG0103
+U 1 1 5CABD795
+P 7475 3150
+F 0 "#FLG0103" H 7475 3225 50  0001 C CNN
+F 1 "PWR_FLAG" H 7475 3323 50  0000 C CNN
+F 2 "" H 7475 3150 50  0001 C CNN
+F 3 "~" H 7475 3150 50  0001 C CNN
+	1    7475 3150
+	1    0    0    -1
+$EndComp
+Connection ~ 7475 3150
+Wire Wire Line
+	7475 3150 7575 3150
+Wire Wire Line
+	3675 4225 3675 4275
+Wire Wire Line
+	4000 4225 3675 4225
+Wire Wire Line
+	4000 4275 4000 4225
+$Comp
+L power:GND #PWR0112
+U 1 1 5CABC5D8
+P 3675 4275
+F 0 "#PWR0112" H 3675 4025 50  0001 C CNN
+F 1 "GND" H 3680 4102 50  0000 C CNN
+F 2 "" H 3675 4275 50  0001 C CNN
+F 3 "" H 3675 4275 50  0001 C CNN
+	1    3675 4275
+	1    0    0    -1
+$EndComp
+$Comp
+L power:PWR_FLAG #FLG0101
+U 1 1 5CABBC7B
+P 4000 4275
+F 0 "#FLG0101" H 4000 4350 50  0001 C CNN
+F 1 "PWR_FLAG" H 4000 4448 50  0000 C CNN
+F 2 "" H 4000 4275 50  0001 C CNN
+F 3 "~" H 4000 4275 50  0001 C CNN
+	1    4000 4275
+	-1   0    0    1
+$EndComp
 $EndSCHEMATC
